Commit message: Version_funcional_gazebo_moviet

File: abb_experimental/abb_irb140_gazebo/urdf/irb140.xacro (robot description, xacro)
@@ -10,2 +10,3 @@
   </joint>
 </robot>
+<!-- Check -->

File: abb_experimental/abb_irb140_gazebo/urdf/irb140_macro.xacro (robot description, xacro)
@@ -5,34 +5,5 @@
   <!-- get base ABB IRB120 model -->
   <xacro:abb_irb140 prefix="${prefix}" />
-  <!-- Gazebo-specific link properties -->
-  <gazebo reference="${prefix}base_link">
-    <material>Gazebo/Orange</material>
-    <turnGravityOff>true</turnGravityOff>
-  </gazebo>
-  <gazebo reference="${prefix}link_1">
-    <material>Gazebo/Orange</material>
-    <turnGravityOff>true</turnGravityOff>
-  </gazebo>
-  <gazebo reference="${prefix}link_2">
-    <material>Gazebo/Orange</material>
-    <turnGravityOff>true</turnGravityOff>
-  </gazebo>
-  <gazebo reference="${prefix}link_3">
-    <material>Gazebo/Orange</material>
-    <turnGravityOff>true</turnGravityOff>
-  </gazebo>
-  <gazebo reference="${prefix}link_4">
-    <material>Gazebo/Orange</material>
-    <turnGravityOff>true</turnGravityOff>
-  </gazebo>
-  <gazebo reference="${prefix}link_5">
-    <material>Gazebo/Orange</material>
-    <turnGravityOff>true</turnGravityOff>
-  </gazebo>
-  <gazebo reference="${prefix}link_6">
-    <material>Gazebo/Black</material>
-    <turnGravityOff>true</turnGravityOff>
-  </gazebo>
-  <!-- transmission list -->
+<!-- transmission list -->
   <transmission name="${prefix}tran1">
     <type>transmission_interface/SimpleTransmission</type>
@@ -90,4 +61,34 @@
   </transmission>
   <!-- end of transmission list -->
+  <!-- Gazebo-specific link properties -->
+  <gazebo reference="${prefix}base_link">
+    <material>Gazebo/Orange</material>
+    <turnGravityOff>true</turnGravityOff>
+  </gazebo>
+  <gazebo reference="${prefix}link_1">
+    <material>Gazebo/Orange</material>
+    <turnGravityOff>true</turnGravityOff>
+  </gazebo>
+  <gazebo reference="${prefix}link_2">
+    <material>Gazebo/Orange</material>
+    <turnGravityOff>true</turnGravityOff>
+  </gazebo>
+  <gazebo reference="${prefix}link_3">
+    <material>Gazebo/Orange</material>
+    <turnGravityOff>true</turnGravityOff>
+  </gazebo>
+  <gazebo reference="${prefix}link_4">
+    <material>Gazebo/Orange</material>
+    <turnGravityOff>true</turnGravityOff>
+  </gazebo>
+  <gazebo reference="${prefix}link_5">
+    <material>Gazebo/Orange</material>
+    <turnGravityOff>true</turnGravityOff>
+  </gazebo>
+  <gazebo reference="${prefix}link_6">
+    <material>Gazebo/Black</material>
+    <turnGravityOff>true</turnGravityOff>
+  </gazebo>
+  <!-- End of Gazebo-specific link properties -->
   <!-- ros_control plugin -->
   <gazebo>

File: abb_experimental/abb_irb140_support/urdf/irb140_macro.xacro (robot description, xacro)
@@ -206,5 +206,5 @@
     <link name="${prefix}tool0"/>
     <!-- end of link list -->
-    <!-- end of joint list -->
+    <!-- tiene pinta que le falta cosas para manejar en Robotestudio-->
     <!-- ROS base_link to ABB World Coordinates transform -->
     <link name="${prefix}base" />
